File: pcb/raspilot.sch (EAGLE design)
At the start: 26 parts, among them IC1 STM32F10XCXT6, K1 PIN20X2, U1 EEPROM-I2CSMD

Commit message: controls
Other:
- note added: "NETFORCE CO. LTD."
- note removed: "FE ROBOTICS CO LTD."
Changed lines of the file:
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@@
 <text x="289.56" y="20.32" size="1.778" layer="94" ratio="15">Drawn by:</text>
 <text x="289.56" y="16.51" size="1.778" layer="94" ratio="15">Checked  by:</text>
-<text x="289.56" y="5.08" size="1.778" layer="94">FE ROBOTICS CO LTD.</text>
+<text x="289.56" y="5.08" size="1.778" layer="94">NETFORCE CO. LTD.</text>
 <text x="309.88" y="20.32" size="1.778" layer="94">David Janssens</text>
 <text x="374.65" y="5.08" size="2.54" layer="94" ratio="10">v0.1</text>
