File: pcb/raspilot.brd (EAGLE design)
At the start: 63 x 54.5 mm, 26 parts, among them IC1 STM32F10XCXT6, K1 PIN20X2, U1 EEPROM-I2CSMD

Commit message: update pcb
Parts:
- moved JP23 5.79 mm to (8.66, 10.3)
- moved JP22 5.79 mm to (8.66, 7.72)
- moved JP21 5.79 mm to (8.66, 5.18)
- moved C4 1.88 mm to (31.9, 18.5)
Routing:
- net +3V3: track 158.0 -> 203.6 mm, vias 7 -> 5
- net GND: track 65.8 -> 25.0 mm
- net PWM4: track 18.6 -> 53.7 mm, vias 1 -> 0
- net PWM6: track 25.5 -> 58.8 mm, vias 1 -> 0
- net LED1: track 62.7 -> 90.1 mm, vias 2 -> 0
- net LED2: track 63.1 -> 88.4 mm
- net USART1_RX: track 57.6 -> 35.7 mm
- net PWM5: track 50.6 -> 30.8 mm, vias 0 -> 1
- net OTHER1: track 57.3 -> 38.6 mm
- net +5V: track 87.3 -> 101.4 mm
- net CAN_L: track 39.8 -> 53.9 mm, vias 1 -> 2
- net PWM3: track 21.4 -> 30.5 mm
- net USART3_RX: track 22.1 -> 30.6 mm, vias 0 -> 1
- net CAN_RX: track 47.6 -> 56.0 mm
- net PWM8: track 20.9 -> 27.3 mm
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Other:
- board text added: "v1.0"
