File: pcb/cellpilot.sch (EAGLE design)
At the start: 26 parts, among them IC1 STM32F10XCXT6, K1 PIN20X2, U1 EEPROM-I2CSMD

Commit message: move connector
Parts:
- removed C11: (no value), adafruit:CPOL-USE2.5-6
Connections:
- net +3V3: no longer C11.+
- net GND: no longer C11.-
Changed lines of the file:
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@@
 <part name="GND7" library="supply1" deviceset="GND" device=""/>
 <part name="GND27" library="supply1" deviceset="GND" device=""/>
-<part name="C11" library="adafruit" deviceset="CPOL-US" device="E2.5-6"/>
-<part name="GND21" library="supply1" deviceset="GND" device=""/>
 <part name="C5" library="SparkFun-Passives" deviceset="CAP" device="0805"/>
 <part name="IC1" library="stm32" deviceset="STM32F10XCXT6" device=""/>
@@
 <instance part="GND7" gate="1" x="40.64" y="121.92"/>
 <instance part="GND27" gate="1" x="83.82" y="165.1"/>
-<instance part="C11" gate="G$1" x="91.44" y="175.26"/>
-<instance part="GND21" gate="1" x="91.44" y="165.1"/>
 <instance part="C5" gate="G$1" x="83.82" y="172.72"/>
 <instance part="IC1" gate="PORTA_L" x="167.64" y="213.36"/>
@@
 </segment>
 <segment>
-<pinref part="GND21" gate="1" pin="GND"/>
-<pinref part="C11" gate="G$1" pin="-"/>
-<wire x1="91.44" y1="167.64" x2="91.44" y2="170.18" width="0.1524" layer="91"/>
-</segment>
-<segment>
 <pinref part="DA1" gate="G$1" pin="GND"/>
 <wire x1="289.56" y1="185.42" x2="294.64" y2="185.42" width="0.1524" layer="91"/>
@@
 <wire x1="35.56" y1="175.26" x2="35.56" y2="180.34" width="0.1524" layer="91"/>
 <pinref part="+3V1" gate="G$1" pin="+3V3"/>
-<pinref part="C11" gate="G$1" pin="+"/>
 <wire x1="78.74" y1="177.8" x2="83.82" y2="177.8" width="0.1524" layer="91"/>
 <pinref part="C5" gate="G$1" pin="1"/>
-<wire x1="83.82" y1="177.8" x2="91.44" y2="177.8" width="0.1524" layer="91"/>
-<junction x="83.82" y="177.8"/>
 <wire x1="78.74" y1="177.8" x2="78.74" y2="193.04" width="0.1524" layer="91"/>
 <wire x1="78.74" y1="193.04" x2="40.64" y2="193.04" width="0.1524" layer="91"/>
